Commit message: NTU-UGV-Version-Arm-Platform

File: tm_description/urdf/tm12x-nominal.urdf (robot description, URDF)
Before this commit: robot tm12x, 11 links, 10 joints
Joints:
- joint shoulder_1_joint: limit lower=-6.283185307179586 upper=6.283185307179586 effort=353 velocity=2.0943951023931953 -> lower=-4.71238898038469 upper=4.71238898038469 effort=353 velocity=2.0943951023931953
- joint shoulder_2_joint: limit lower=-6.283185307179586 upper=6.283185307179586 effort=353 velocity=2.0943951023931953 -> lower=-3.141592653589793 upper=3.141592653589793 effort=353 velocity=2.0943951023931953
- joint wrist_1_joint: limit lower=-6.283185307179586 upper=6.283185307179586 effort=54 velocity=3.141592653589793 -> lower=-3.141592653589793 upper=3.141592653589793 effort=54 velocity=3.141592653589793
- joint wrist_2_joint: limit lower=-6.283185307179586 upper=6.283185307179586 effort=54 velocity=3.141592653589793 -> lower=-3.141592653589793 upper=3.141592653589793 effort=54 velocity=3.141592653589793
- joint wrist_3_joint: limit lower=-6.283185307179586 upper=6.283185307179586 effort=54 velocity=3.141592653589793 -> lower=-4.71238898038469 upper=4.71238898038469 effort=54 velocity=3.141592653589793

File: tm_description/urdf/tm14x-nominal.urdf (robot description, URDF)
Before this commit: robot tm14x, 11 links, 10 joints
Joints:
- joint shoulder_1_joint: limit lower=-6.283185307179586 upper=6.283185307179586 effort=353 velocity=2.0943951023931953 -> lower=-4.71238898038469 upper=4.71238898038469 effort=353 velocity=2.0943951023931953
- joint shoulder_2_joint: limit lower=-6.283185307179586 upper=6.283185307179586 effort=353 velocity=2.0943951023931953 -> lower=-3.141592653589793 upper=3.141592653589793 effort=353 velocity=2.0943951023931953
- joint wrist_1_joint: limit lower=-6.283185307179586 upper=6.283185307179586 effort=54 velocity=2.6179938779914944 -> lower=-3.141592653589793 upper=3.141592653589793 effort=54 velocity=2.6179938779914944
- joint wrist_2_joint: limit lower=-6.283185307179586 upper=6.283185307179586 effort=54 velocity=2.6179938779914944 -> lower=-3.141592653589793 upper=3.141592653589793 effort=54 velocity=2.6179938779914944
- joint wrist_3_joint: limit lower=-6.283185307179586 upper=6.283185307179586 effort=54 velocity=3.141592653589793 -> lower=-4.71238898038469 upper=4.71238898038469 effort=54 velocity=3.141592653589793

File: tm_description/urdf/tm5x-700-nominal.urdf (robot description, URDF)
Before this commit: robot tm5x-700, 11 links, 10 joints
Joints:
- joint shoulder_1_joint: limit lower=-6.283185307179586 upper=6.283185307179586 effort=157 velocity=3.141592653589793 -> lower=-4.71238898038469 upper=4.71238898038469 effort=157 velocity=3.141592653589793
- joint shoulder_2_joint: limit lower=-6.283185307179586 upper=6.283185307179586 effort=157 velocity=3.141592653589793 -> lower=-3.141592653589793 upper=3.141592653589793 effort=157 velocity=3.141592653589793
- joint wrist_1_joint: limit lower=-6.283185307179586 upper=6.283185307179586 effort=43 velocity=3.9269908169872414 -> lower=-3.141592653589793 upper=3.141592653589793 effort=43 velocity=3.9269908169872414
- joint wrist_2_joint: limit lower=-6.283185307179586 upper=6.283185307179586 effort=43 velocity=3.9269908169872414 -> lower=-3.141592653589793 upper=3.141592653589793 effort=43 velocity=3.9269908169872414
- joint wrist_3_joint: limit lower=-6.283185307179586 upper=6.283185307179586 effort=43 velocity=3.9269908169872414 -> lower=-4.71238898038469 upper=4.71238898038469 effort=43 velocity=3.9269908169872414

File: tm_description/urdf/tm5x-900-nominal.urdf (robot description, URDF)
Before this commit: robot tm5x-900, 11 links, 10 joints
Joints:
- joint shoulder_1_joint: limit lower=-6.283185307179586 upper=6.283185307179586 effort=157 velocity=3.141592653589793 -> lower=-4.71238898038469 upper=4.71238898038469 effort=157 velocity=3.141592653589793
- joint shoulder_2_joint: limit lower=-6.283185307179586 upper=6.283185307179586 effort=157 velocity=3.141592653589793 -> lower=-3.141592653589793 upper=3.141592653589793 effort=157 velocity=3.141592653589793
- joint wrist_1_joint: limit lower=-6.283185307179586 upper=6.283185307179586 effort=43 velocity=3.9269908169872414 -> lower=-3.141592653589793 upper=3.141592653589793 effort=43 velocity=3.9269908169872414
- joint wrist_2_joint: limit lower=-6.283185307179586 upper=6.283185307179586 effort=43 velocity=3.9269908169872414 -> lower=-3.141592653589793 upper=3.141592653589793 effort=43 velocity=3.9269908169872414
- joint wrist_3_joint: limit lower=-6.283185307179586 upper=6.283185307179586 effort=43 velocity=3.9269908169872414 -> lower=-4.71238898038469 upper=4.71238898038469 effort=43 velocity=3.9269908169872414

File: tm_description/xacro/macro.tm12x-nominal.urdf.xacro (robot description, xacro)
@@ -3,10 +3,10 @@
   <xacro:include filename="$(find tm_description)/xacro/macro.inertial.xacro" />
   <xacro:macro name="tm12x" params="ns prefix color:=none format:=obj
-    shoulder_1_joint_lower_limit:=${radians(-360)}    shoulder_1_joint_upper_limit:=${radians(360)}
-    shoulder_2_joint_lower_limit:=${radians(-360)}    shoulder_2_joint_upper_limit:=${radians(360)}
+    shoulder_1_joint_lower_limit:=${radians(-270)}    shoulder_1_joint_upper_limit:=${radians(270)}
+    shoulder_2_joint_lower_limit:=${radians(-180)}    shoulder_2_joint_upper_limit:=${radians(180)}
     elbow_joint_lower_limit:=${radians(-166)}    elbow_joint_upper_limit:=${radians(166)}
-    wrist_1_joint_lower_limit:=${radians(-360)}    wrist_1_joint_upper_limit:=${radians(360)}
-    wrist_2_joint_lower_limit:=${radians(-360)}    wrist_2_joint_upper_limit:=${radians(360)}
-    wrist_3_joint_lower_limit:=${radians(-360)}    wrist_3_joint_upper_limit:=${radians(360)}
+    wrist_1_joint_lower_limit:=${radians(-180)}    wrist_1_joint_upper_limit:=${radians(180)}
+    wrist_2_joint_lower_limit:=${radians(-180)}    wrist_2_joint_upper_limit:=${radians(180)}
+    wrist_3_joint_lower_limit:=${radians(-270)}    wrist_3_joint_upper_limit:=${radians(270)}
     shoulder_1_joint_velocity_limit:=${radians(120)}
     shoulder_2_joint_velocity_limit:=${radians(120)}

File: tm_description/xacro/macro.tm5-900-nominal.urdf.xacro (robot description, xacro)
@@ -280,4 +280,29 @@
     <origin rpy="0.000000 0.000000 0.000000" xyz="0.000000 0.000000 0.000000" />
   </joint>
+      <link name="${prefix}realsense_fixture">
+      <visual>
+        <geometry>
+          <mesh filename="package://tm_description/meshes/tm5-900/visual/realsense_fixture.${format}" />
+        </geometry>
+        <material name="${color}" />
+      </visual>
+      <collision>
+        <geometry>
+          <mesh filename="package://tm_description/meshes/tm5-900/collision/TM_Realsense_Rviz_Collision_meter.stl" />
+        </geometry>
+      </collision>
+    </link>
+    <joint name="${prefix}flange_link-realsense" type="fixed">
+      <parent link="${prefix}flange_link" />
+      <child link="${prefix}realsense_fixture" />
+      <origin rpy="-0.0 0.0 -3.14" xyz="0.031 0.12422165 0.05114026" />
+      <!-- <origin rpy="-0.0403348 0.01678710 -3.1261744" xyz="0.031 0.12422165 0.05114026" /> -->
+    </joint>
+    <link name="${prefix}camera_link"/>
+    <joint name="${prefix}realsense_optical_camera_center" type="fixed">
+      <parent link="${prefix}realsense_fixture" />
+      <child link="${prefix}camera_link" />
+      <origin rpy="-0.0   -1.57    1.57" xyz="0.0148 0.0001 0.0002" />
+    </joint>
 <!--LinkDescription-->
   </xacro:macro>

File: tm_description/xacro/macro.tm5x-700-nominal.urdf.xacro (robot description, xacro)
@@ -3,10 +3,10 @@
   <xacro:include filename="$(find tm_description)/xacro/macro.inertial.xacro" />
   <xacro:macro name="tm5x-700" params="ns prefix color:=none format:=obj
-    shoulder_1_joint_lower_limit:=${radians(-360)}    shoulder_1_joint_upper_limit:=${radians(360)}
-    shoulder_2_joint_lower_limit:=${radians(-360)}    shoulder_2_joint_upper_limit:=${radians(360)}
+    shoulder_1_joint_lower_limit:=${radians(-270)}    shoulder_1_joint_upper_limit:=${radians(270)}
+    shoulder_2_joint_lower_limit:=${radians(-180)}    shoulder_2_joint_upper_limit:=${radians(180)}
     elbow_joint_lower_limit:=${radians(-155)}    elbow_joint_upper_limit:=${radians(155)}
-    wrist_1_joint_lower_limit:=${radians(-360)}    wrist_1_joint_upper_limit:=${radians(360)}
-    wrist_2_joint_lower_limit:=${radians(-360)}    wrist_2_joint_upper_limit:=${radians(360)}
-    wrist_3_joint_lower_limit:=${radians(-360)}    wrist_3_joint_upper_limit:=${radians(360)}
+    wrist_1_joint_lower_limit:=${radians(-180)}    wrist_1_joint_upper_limit:=${radians(180)}
+    wrist_2_joint_lower_limit:=${radians(-180)}    wrist_2_joint_upper_limit:=${radians(180)}
+    wrist_3_joint_lower_limit:=${radians(-270)}    wrist_3_joint_upper_limit:=${radians(270)}
     shoulder_1_joint_velocity_limit:=${radians(180)}
     shoulder_2_joint_velocity_limit:=${radians(180)}

File: tm_description/xacro/macro.tm5x-900-nominal.urdf.xacro (robot description, xacro)
@@ -3,10 +3,10 @@
   <xacro:include filename="$(find tm_description)/xacro/macro.inertial.xacro" />
   <xacro:macro name="tm5x-900" params="ns prefix color:=none format:=obj
-    shoulder_1_joint_lower_limit:=${radians(-360)}    shoulder_1_joint_upper_limit:=${radians(360)}
-    shoulder_2_joint_lower_limit:=${radians(-360)}    shoulder_2_joint_upper_limit:=${radians(360)}
+    shoulder_1_joint_lower_limit:=${radians(-270)}    shoulder_1_joint_upper_limit:=${radians(270)}
+    shoulder_2_joint_lower_limit:=${radians(-180)}    shoulder_2_joint_upper_limit:=${radians(180)}
     elbow_joint_lower_limit:=${radians(-155)}    elbow_joint_upper_limit:=${radians(155)}
-    wrist_1_joint_lower_limit:=${radians(-360)}    wrist_1_joint_upper_limit:=${radians(360)}
-    wrist_2_joint_lower_limit:=${radians(-360)}    wrist_2_joint_upper_limit:=${radians(360)}
-    wrist_3_joint_lower_limit:=${radians(-360)}    wrist_3_joint_upper_limit:=${radians(360)}
+    wrist_1_joint_lower_limit:=${radians(-180)}    wrist_1_joint_upper_limit:=${radians(180)}
+    wrist_2_joint_lower_limit:=${radians(-180)}    wrist_2_joint_upper_limit:=${radians(180)}
+    wrist_3_joint_lower_limit:=${radians(-270)}    wrist_3_joint_upper_limit:=${radians(270)}
     shoulder_1_joint_velocity_limit:=${radians(180)}
     shoulder_2_joint_velocity_limit:=${radians(180)}
