Commit message: update for ntu-greenhouse

File: tm_description/xacro/macro.tm5-900-nominal-614.urdf.xacro (robot description, xacro)
@@ -366,21 +366,5 @@
       <origin rpy="0.000000 0.000000 0.000000" xyz="0.000000 0.000000 0.000000" />
     </joint>
-    <link name="${prefix}tool0" >
-      <!-- <visual>
-        <origin xyz="0 0 0.155" rpy="0 0 0" />
-      <geometry>
-       	<cylinder radius="0.01" length="0.31"/>
-      </geometry>
-      <material name="white">
-        <color rgba="0.3 1 1 1"/>
-      </material>
-      </visual>
-      <collision>
-        <origin xyz="0 0 0.19" rpy="0 0 0"/>
-        <geometry>
-          <cylinder radius="0.03" length="0.24"/>
-        </geometry>
-      </collision> -->
-    </link>
+    <link name="${prefix}tool0"/>
     <joint name="${prefix}flange_link-tool0" type="fixed">
       <parent link="${prefix}flange_link" />
@@ -388,10 +372,4 @@
       <origin rpy="0.000000 0.000000 0.000000" xyz="0.000000 0.000000 0.000000" />
     </joint>
-    <!-- <link name="${prefix}gripper" />
-    <joint name="${prefix}tool0-gripper" type="fixed">
-      <parent link="${prefix}tool0" />
-      <child link="${prefix}gripper" />
-      <origin rpy="0.000000 0.000000 0.000000" xyz="0.000000 0.000000 0.31" />
-    </joint> -->
     <link name="${prefix}realsense_fixture">
       <visual>
@@ -411,5 +389,4 @@
       <child link="${prefix}realsense_fixture" />
       <origin rpy="-0.0 0.0 -3.14" xyz="0.031 0.12422165 0.05114026" />
-      <!-- <origin rpy="-0.0403348 0.01678710 -3.1261744" xyz="0.031 0.12422165 0.05114026" /> -->
     </joint>
     <link name="${prefix}camera_link"/>

File: tm_description/xacro/macro.tm5-900-nominal.urdf.xacro (robot description, xacro)
@@ -280,29 +280,4 @@
     <origin rpy="0.000000 0.000000 0.000000" xyz="0.000000 0.000000 0.000000" />
   </joint>
-      <link name="${prefix}realsense_fixture">
-      <visual>
-        <geometry>
-          <mesh filename="package://tm_description/meshes/tm5-900/visual/realsense_fixture.${format}" />
-        </geometry>
-        <material name="${color}" />
-      </visual>
-      <collision>
-        <geometry>
-          <mesh filename="package://tm_description/meshes/tm5-900/collision/TM_Realsense_Rviz_Collision_meter.stl" />
-        </geometry>
-      </collision>
-    </link>
-    <joint name="${prefix}flange_link-realsense" type="fixed">
-      <parent link="${prefix}flange_link" />
-      <child link="${prefix}realsense_fixture" />
-      <origin rpy="-0.0 0.0 -3.14" xyz="0.031 0.12422165 0.05114026" />
-      <!-- <origin rpy="-0.0403348 0.01678710 -3.1261744" xyz="0.031 0.12422165 0.05114026" /> -->
-    </joint>
-    <link name="${prefix}camera_link"/>
-    <joint name="${prefix}realsense_optical_camera_center" type="fixed">
-      <parent link="${prefix}realsense_fixture" />
-      <child link="${prefix}camera_link" />
-      <origin rpy="-0.0   -1.57    1.57" xyz="0.0148 0.0001 0.0002" />
-    </joint>
 <!--LinkDescription-->
   </xacro:macro>

File: tm_description/xacro/tm5-900-614.urdf.xacro (robot description, xacro)
@@ -16,4 +16,5 @@
   <xacro:tmr_transmission prefix="$(arg prefix)" hw_iface="$(arg trans_hw_iface)" />
   <xacro:tmr_materials/>
+  sss
   <!-- Arm -->
   <xacro:property name="color" value="$(arg color)"/>
